File: Morphex-PCB/Morphex-PCB.kicad_pcb (KiCad board)
At the start: 4 copper layers, 76.2 x 58.5 mm, 37 parts, among them IC1 TXB0108PWR, IC2 NC7WZ241K8X, J1 Main Terminal, U1 DEV-16771, U2 NRF24, U3 BNO055

Commit message: update pcb
Parts:
- added 3.3V: Conn_01x03_Pin, Connector_PinHeader_2.54mm:PinHeader_1x03_P2.54mm_Vertical, F.Cu at (185.1, 85.0)
- added 5V: Conn_01x03_Pin, Connector_PinHeader_2.54mm:PinHeader_1x03_P2.54mm_Vertical, F.Cu at (185.1, 89.7)
- added J2: SERIAL2, Connector_PinHeader_2.54mm:PinHeader_1x02_P2.54mm_Vertical, F.Cu at (161.9, 83.5)
- added J3: SERIAL7, Connector_PinHeader_2.54mm:PinHeader_1x02_P2.54mm_Vertical, F.Cu at (164.7, 83.5)
- added J4: CAN_SERIAL3, Connector_PinHeader_2.54mm:PinHeader_1x02_P2.54mm_Vertical, F.Cu at (167.4, 83.5)
- added J5: SERIAL8, Connector_PinHeader_2.54mm:PinHeader_1x02_P2.54mm_Vertical, F.Cu at (170.2, 83.5)
- added R4: 10K, Resistor_SMD:R_0603_1608Metric_Pad0.98x0.95mm_HandSolder, F.Cu at (184.0, 81.1)
- added SW1: Push_Button, Button_Switch_THT:SW_PUSH_6mm, F.Cu at (176.8, 81.2)
- 33R: renamed from 33R1; footprint 33R:DPAK_STM -> footprints:DPAK_STM
- 50R: renamed from 50R1; footprint 33R:DPAK_STM -> footprints:DPAK_STM
- Main Terminal: renamed from J1
- moved C9 86.9 mm to (182.0, 103.6), turned to 90 degrees
- moved C6 85.5 mm to (178.5, 104.8), turned to 180 degrees
- moved R3 84.9 mm to (182.0, 97.5), turned to -90 degrees
- moved R2 81.1 mm to (178.2, 95.2), turned to 180 degrees
- moved C8 78.5 mm to (174.0, 102.6), turned to -90 degrees
- moved C7 77.4 mm to (171.8, 102.2), turned to 90 degrees
- moved IC2 69.4 mm to (155.2, 98.2)
- moved IC1 66.0 mm to (145.8, 100.2), turned to 0 degrees
- moved 33R 54.8 mm to (188.5, 115.2), turned to 180 degrees
- moved C5 54.5 mm to (148.0, 94.8)
- moved 50R 54.1 mm to (188.5, 100.5), turned to 180 degrees
- moved C3 53.9 mm to (148.2, 86.4), turned to -90 degrees
- moved C4 53.8 mm to (140.0, 104.2), turned to -90 degrees
- moved R1 48.7 mm to (143.0, 105.2)
- moved C1 32.4 mm to (121.7, 83.7)
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Connections:
- U1 pad 14: unconnected-(U1-A0-Pad14) -> /BNO_RESET
- U1 pad 15: unconnected-(U1-A1-Pad15) -> /BNO_INT
- U1 pad 28: unconnected-(U1-RX7-Pad28) -> /rx7
- U1 pad 29: unconnected-(U1-TX7-Pad29) -> /tx7
- U1 pad 30: unconnected-(U1-CRX3-Pad30) -> /crx3
- U1 pad 31: unconnected-(U1-CTX3-Pad31) -> /ctx3
- U1 pad 34: unconnected-(U1-RX8-Pad34) -> /rx8
- U1 pad 35: unconnected-(U1-TX8-Pad35) -> /tx8
- U1 pad 37: unconnected-(U1-CS3-Pad37) -> /BUTTON_PIN
- U1 pad 7: /BNO_RESET -> /rx2
- U1 pad 8: /BNO_INT -> /tx2
Routing:
- net GND: track 0.00 -> 213.9 mm, vias 0 -> 2
- net +3.3V: track 0.00 -> 175.0 mm, vias 0 -> 8
- net +5V: track 0.00 -> 140.3 mm, vias 0 -> 8
- net /from_servo: track 0.00 -> 135.3 mm, vias 0 -> 1
- net VCC: track 0.00 -> 89.1 mm, vias 0 -> 2
- net /rx2: track 0.00 -> 66.5 mm, vias 0 -> 1
- net /tx2: track 0.00 -> 66.2 mm, vias 0 -> 1
- net /NRF_CS: track 0.00 -> 56.9 mm, vias 0 -> 1
- net /NRF_MOSI: track 0.00 -> 54.6 mm, vias 0 -> 2
- net /BNO_INT: track 0.00 -> 51.3 mm, vias 0 -> 2
- net /SDA: track 0.00 -> 43.7 mm, vias 0 -> 1
- net /SCL: track 0.00 -> 43.2 mm, vias 0 -> 2
- net /NRF_MISO: track 0.00 -> 41.6 mm, vias 0 -> 1
- net /BNO_RESET: track 0.00 -> 40.8 mm, vias 0 -> 4
- net /ctx3: track 0.00 -> 36.4 mm, vias 0 -> 3
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- added copper zone on B.Cu, net GND
- added copper zone on In2.Cu, net GND
- added copper zone on F.Cu, net VCC
- added copper zone on In1.Cu, net VCC
Other:
- board text added: "CAN"
- board text added: "RX"
- board text added: "S2"
- board text added: "S3"
- board text added: "S7"
- board text added: "S8"
- board text added: "SERIAL"
- board text added: "TX"
