File: Morphex-PCB/Morphex-PCB.kicad_pcb (KiCad board)
At the start: 4 copper layers, 76.2 x 58.5 mm, 45 parts, among them IC1 TXB0108PWR, IC2 NC7WZ241K8X, J2 SERIAL2, J3 SERIAL7, J4 CAN_SERIAL3, J5 SERIAL8, SW1 Push_Button, U1 DEV-16771, U2 NRF24, U3 BNO055

Commit message: update pcb
Other:
- board text added: "Jirakorn Sukmee's Teensy 4.1 Hexapod PCB"
Changed lines of the file:
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@@
 		(allow_soldermask_bridges_in_footprints no)
 		(pcbplotparams
-			(layerselection 0x00010fc_ffffffff)
+			(layerselection 0x00010f4_ffffffff)
 			(plot_on_all_layers_selection 0x0000000_00000000)
 			(disableapertmacros no)
@@
 			(outputformat 1)
 			(mirror no)
-			(drillshape 1)
+			(drillshape 0)
 			(scaleselection 1)
-			(outputdirectory "")
+			(outputdirectory "Gerber/")
 		)
 	)
@@
 		(tags "mounting hole 3.2mm no annular m3")
 		(property "Reference" "H1"
-			(at 0 -4.2 0)
+			(at 0 -3.9 180)
 			(layer "F.SilkS")
 			(effects
@@
 			)
 			(justify left bottom)
+		)
+	)
+	(gr_text "Jirakorn Sukmee's \nTeensy 4.1 \nHexapod PCB"
+		(at 172.8 73.8 180)
+		(layer "F.SilkS")
+		(effects
+			(font
+				(size 1 1)
+				(thickness 0.15)
+			)
+			(justify left bottom)
