File: Morphex-PCB/Morphex-PCB.kicad_pcb (KiCad board)
At the start: 4 copper layers, 76.2 x 58.5 mm, 45 parts, among them IC1 TXB0108PWR, IC2 NC7WZ241K8X, J2 SERIAL2, J3 SERIAL7, J4 CAN_SERIAL3, J5 SERIAL8, SW1 Push_Button, U1 DEV-16771, U2 NRF24, U3 BNO055

Commit message: fixed PCB
Parts:
- 33R1: renamed from 33R; footprint footprints:DPAK_STM -> 33R:DPAK_STM
- 50R1: renamed from 50R; footprint footprints:DPAK_STM -> 33R:DPAK_STM
- C1, C4, C5, C6, C7, C9: footprint Capacitor_SMD:C_0805_2012Metric_Pad1.18x1.45mm_HandSolder -> Capacitor_SMD:C_0603_1608Metric_Pad1.08x0.95mm_HandSolder
- renumbered 5V to +5V
Connections:
- servo1 pad 1: VCC -> GND
- servo1 pad 2: GND -> VCC
- servo10 pad 1: VCC -> GND
- servo10 pad 2: GND -> VCC
- servo11 pad 1: VCC -> GND
- servo11 pad 2: GND -> VCC
- servo12 pad 1: VCC -> GND
- servo12 pad 2: GND -> VCC
- servo13 pad 1: VCC -> GND
- servo13 pad 2: GND -> VCC
- servo2 pad 1: VCC -> GND
- servo2 pad 2: GND -> VCC
- servo3 pad 1: VCC -> GND
- servo3 pad 2: GND -> VCC
- servo4 pad 1: VCC -> GND
- servo4 pad 2: GND -> VCC
- servo5 pad 1: VCC -> GND
- servo5 pad 2: GND -> VCC
- servo6 pad 1: VCC -> GND
- servo6 pad 2: GND -> VCC
- servo7 pad 1: VCC -> GND
- servo7 pad 2: GND -> VCC
- servo8 pad 1: VCC -> GND
- servo8 pad 2: GND -> VCC
- servo9 pad 1: VCC -> GND
- servo9 pad 2: GND -> VCC
Routing:
- net GND: track 357.8 -> 358.4 mm
Other:
- board text added: "33R"
- board text added: "50R"

Commit message: updated pcb
Parts:
- added GND: Conn_01x03_Pin, Connector_PinHeader_2.54mm:PinHeader_1x03_P2.54mm_Vertical, F.Cu at (185.4, 84.5)
- moved 3.3V 2.61 mm to (185.4, 87.6)
- moved +5V 1.08 mm to (185.4, 90.7)
Routing:
- net +3.3V: track 192.7 -> 249.3 mm
- net VCC: track 89.2 -> 87.8 mm
- net +5V: track 140.3 -> 141.1 mm
Other:
- board text added: "+"
- board text added: "-"
