File: Morphex-PCB/Morphex-PCB.kicad_sch (KiCad schematic)
At the start: 26 parts, among them IC1 TXB0108PWR, IC2 NC7WZ241K8X, J1 Main Terminal, J10 Conn_01x03_Socket, J11 Conn_01x03_Socket, J12 Conn_01x03_Socket, J13 Conn_01x03_Socket, J2 Conn_01x03_Socket, J3 Conn_01x03_Socket, J4 Conn_01x03_Socket, J5 Conn_01x03_Socket, J6 Conn_01x03_Socket, J7 Conn_01x03_Socket, J8 Conn_01x03_Socket, J9 Conn_01x03_Socket, U1 DEV-16771, U2 NRF24, U3 BNO055

Commit message: update pcb
Parts:
- added servo13: Conn_01x03_Socket, symbol Connector:Conn_01x03_Socket
- renumbered J3 to servo1, J10 to servo10, J11 to servo11, J13 to servo12, J2 to servo2, J4 to servo3, J5 to servo4, J6 to servo5, J12 to servo6, J7 to servo7, J8 to servo8, J9 to servo9
Other:
- company: (none) -> Jirakorn Sukmee
- title: (none) -> Teensy 4.1 Hexapod PCB 
- moved on the sheet: C3, CR1, CR2, J1, U2, U3, servo1, servo10, servo11, servo12, servo2, servo3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

Commit message: updated pcb
Parts:
- added C6, C7, C9: 0.1uF, Capacitor_SMD:C_0805_2012Metric_Pad1.18x1.45mm_HandSolder, symbol Device:C_Small
- added C8: 0.0068uF, Capacitor_SMD:C_0603_1608Metric_Pad1.08x0.95mm_HandSolder, symbol Device:C_Small
- added H1, H2, H3, H4: MountingHole, MountingHole:MountingHole_3.2mm_M3, symbol Mechanical:MountingHole
- added R2, R3: 10K, Resistor_SMD:R_0603_1608Metric_Pad0.98x0.95mm_HandSolder, symbol Device:R
- C1, C2, C3, C4, C5: footprint (none) -> Capacitor_SMD:C_0805_2012Metric_Pad1.18x1.45mm_HandSolder
- J1: footprint (none) -> TerminalBlock_Phoenix:TerminalBlock_Phoenix_MKDS-1,5-2-5.08_1x02_P5.08mm_Horizontal
- R1: footprint (none) -> Resistor_SMD:R_0603_1608Metric_Pad0.98x0.95mm_HandSolder
- servo1, servo10, servo11, servo12, servo13, servo2, servo3, servo4, servo5, servo6, servo7, servo8, servo9: footprint (none) -> Connector_JST:JST_PH_B3B-PH-K_1x03_P2.00mm_Vertical
- renumbered CR1 to 33R1, CR2 to 50R1
Connections:
- net to_servo is gone; now on net from_servo: IC2.6 (Y1)
- net +3.3V: now also U3.28 (VDDIO), U3.3 (VDD), C6.2, C7.1, C8.2, R2.1, R3.1
- net +5V: now also U1.VIN; no longer U1.5V
- net GND: now also U1.GND1 (GND), U1.GND2 (GND), U1.GND3 (GND), U1.GND4 (GND), U1.GND5 (GND), U1.USB_GND1 (USB_GND), U1.USB_GND2 (USB_GND), U3.15 (GNDIO), U3.16 (GNDIO), U3.17 (COM3), U3.18 (COM2), U3.2 (GND), U3.25 (GNDIO), U3.5 (PS1), U3.6 (PS0), servo1.2 (Pin_2), servo10.2 (Pin_2), servo11.2 (Pin_2), servo12.2 (Pin_2), servo13.2 (Pin_2), servo2.2 (Pin_2), servo3.2 (Pin_2), servo4.2 (Pin_2), servo5.2 (Pin_2), servo6.2 (Pin_2), servo7.2 (Pin_2), servo8.2 (Pin_2), servo9.2 (Pin_2), C6.1, C7.2, C8.1, C9.1
- net VCC: now also servo1.1 (Pin_1), servo10.1 (Pin_1), servo11.1 (Pin_1), servo12.1 (Pin_1), servo13.1 (Pin_1), servo2.1 (Pin_1), servo3.1 (Pin_1), servo4.1 (Pin_1), servo5.1 (Pin_1), servo6.1 (Pin_1), servo7.1 (Pin_1), servo8.1 (Pin_1), servo9.1 (Pin_1)
- net from_servo: now also servo1.3 (Pin_3), servo10.3 (Pin_3), servo11.3 (Pin_3), servo12.3 (Pin_3), servo13.3 (Pin_3), servo2.3 (Pin_3), servo3.3 (Pin_3), servo4.3 (Pin_3), servo5.3 (Pin_3), servo6.3 (Pin_3), servo7.3 (Pin_3), servo8.3 (Pin_3), servo9.3 (Pin_3)
- net servo_dir: now also U1.41 (A17); no longer U1.40 (A16)
- net NRF_CS: now reaches U1.10 (CS1)
- net NRF_CS: now also U2.4 (~{CSN})
- net NRF_MOSI: now reaches U1.11 (MOSI)
- net NRF_MOSI: now also U2.6 (MOSI)
- net NRF_MISO: now reaches U1.12 (MISO)
- net NRF_MISO: now also U2.7 (MISO)
- net NRF_SCK: now reaches U1.13 (SCK)
- net NRF_SCK: now also U2.5 (SCK)
- net SDA: now reaches U1.18 (A4)
- net SDA: now also U3.20 (COM0)
- net SCL: now reaches U1.19 (A5)
- net SCL: now also U3.19 (COM1)
- net BNO_RESET: now reaches U1.7 (RX2)
- net BNO_RESET: now also U3.11 (~{RESET}), R3.2
- net BNO_INT: now reaches U1.8 (TX2)
- net BNO_INT: now also U3.14 (INT)
- net NRF_CE: now reaches U2.3 (CE)
- net NRF_CE: now also U1.40 (A16)
- net at U3.4 (~{BOOT_LOAD_PIN}): now also R2.2
- net at U3.9 (CAP): now also C9.2
Other:
- moved on the sheet: 33R1, 50R1, C1, C2, C3, C4, C5, IC1, IC2, J1, R1, U2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

Commit message: update pcb
Parts:
- added +5V1, 3.3V1: Conn_01x03_Pin, Connector_PinHeader_2.54mm:PinHeader_1x03_P2.54mm_Vertical, symbol Connector:Conn_01x03_Pin
- added J2: SERIAL2, Connector_PinHeader_2.54mm:PinHeader_1x02_P2.54mm_Vertical, symbol Connector:Conn_01x02_Pin
- added J3: SERIAL7, Connector_PinHeader_2.54mm:PinHeader_1x02_P2.54mm_Vertical, symbol Connector:Conn_01x02_Pin
- added J4: CAN_SERIAL3, Connector_PinHeader_2.54mm:PinHeader_1x02_P2.54mm_Vertical, symbol Connector:Conn_01x02_Pin
- added J5: SERIAL8, Connector_PinHeader_2.54mm:PinHeader_1x02_P2.54mm_Vertical, symbol Connector:Conn_01x02_Pin
- added R4: 10K, Resistor_SMD:R_0603_1608Metric_Pad0.98x0.95mm_HandSolder, symbol Device:R
- added SW1: Push_Button, Button_Switch_THT:SW_PUSH_6mm, symbol Switch:SW_Push
Connections:
- net +3.3V: now also 3.3V1.1 (Pin_1), 3.3V1.2 (Pin_2), 3.3V1.3 (Pin_3)
- net +5V: now also +5V1.1 (Pin_1), +5V1.2 (Pin_2), +5V1.3 (Pin_3)
- net BNO_INT: now also U1.15 (A1); no longer U1.8 (TX2)
- net BNO_RESET: now also U1.14 (A0); no longer U1.7 (RX2)
- net GND: now also R4.2
- net rx7: now reaches U1.28 (RX7)
- net rx7: now also J3.2 (Pin_2)
- net tx7: now reaches U1.29 (TX7)
- net tx7: now also J3.1 (Pin_1)
- net crx3: now reaches U1.30 (CRX3)
- net crx3: now also J4.2 (Pin_2)
- net ctx3: now reaches U1.31 (CTX3)
- net ctx3: now also J4.1 (Pin_1)
- net rx8: now reaches U1.34 (RX8)
- net rx8: now also J5.2 (Pin_2)
- net tx8: now reaches U1.35 (TX8)
- net tx8: now also J5.1 (Pin_1)
- net BUTTON_PIN: now reaches U1.37 (CS3)
- net BUTTON_PIN: now also SW1.1
- new net: R4.1, SW1.2
- new net rx2: J2.2 (Pin_2), U1.7 (RX2)
- new net tx2: J2.1 (Pin_1), U1.8 (TX2)
Other:
- moved on the sheet: 33R1, 50R1, C1, C2, C3, C4, C5, C6, C7, C8, C9, IC1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

Commit message: fixed PCB
Parts:
- C1, C4, C5, C6, C7, C9: footprint Capacitor_SMD:C_0805_2012Metric_Pad1.18x1.45mm_HandSolder -> Capacitor_SMD:C_0603_1608Metric_Pad1.08x0.95mm_HandSolder
Connections:
- net GND: now also servo1.1 (Pin_1), servo10.1 (Pin_1), servo11.1 (Pin_1), servo12.1 (Pin_1), servo13.1 (Pin_1), servo2.1 (Pin_1), servo3.1 (Pin_1), servo4.1 (Pin_1), servo5.1 (Pin_1), servo6.1 (Pin_1), servo7.1 (Pin_1), servo8.1 (Pin_1), servo9.1 (Pin_1); no longer servo1.2 (Pin_2), servo10.2 (Pin_2), servo11.2 (Pin_2), servo12.2 (Pin_2), servo13.2 (Pin_2), servo2.2 (Pin_2), servo3.2 (Pin_2), servo4.2 (Pin_2), servo5.2 (Pin_2), servo6.2 (Pin_2), servo7.2 (Pin_2), servo8.2 (Pin_2), servo9.2 (Pin_2)
- net VCC: now also servo1.2 (Pin_2), servo10.2 (Pin_2), servo11.2 (Pin_2), servo12.2 (Pin_2), servo13.2 (Pin_2), servo2.2 (Pin_2), servo3.2 (Pin_2), servo4.2 (Pin_2), servo5.2 (Pin_2), servo6.2 (Pin_2), servo7.2 (Pin_2), servo8.2 (Pin_2), servo9.2 (Pin_2); no longer servo1.1 (Pin_1), servo10.1 (Pin_1), servo11.1 (Pin_1), servo12.1 (Pin_1), servo13.1 (Pin_1), servo2.1 (Pin_1), servo3.1 (Pin_1), servo4.1 (Pin_1), servo5.1 (Pin_1), servo6.1 (Pin_1), servo7.1 (Pin_1), servo8.1 (Pin_1), servo9.1 (Pin_1)

Commit message: updated pcb
Parts:
- added GND1: Conn_01x03_Pin, Connector_PinHeader_2.54mm:PinHeader_1x03_P2.54mm_Vertical, symbol Connector:Conn_01x03_Pin
Connections:
- net GND: now also GND1.1 (Pin_1), GND1.2 (Pin_2), GND1.3 (Pin_3)
