File: PCB-Teensy4.0/Teensy4.0PCB/Teensy4.0PCB.kicad_pcb (KiCad board)
At the start: 4 copper layers, 76 x 58 mm, 53 parts, among them IC1 TXB0108PWR, IC2 NC7WZ241K8X, J1 Conn_01x04_Pin, J2 Conn_01x04_Pin, U1 Teensy4.0, U2 NRF24, U3 BNO055

Commit message: updated teensy's PCB
Routing:
- added copper zone on B.Cu, net GND
- added copper zone on F.Cu, net GND
- removed copper zone on F.Cu, net VCC
Changed lines of the file:
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@@
 		(tags "Through hole pin header THT 1x03 2.54mm single row")
 		(property "Reference" "3.3V1"
-			(at 0 -2.46 360)
+			(at 0 -2.46 0)
 			(layer "F.SilkS")
 			(effects
@@
 		)
 		(property "Value" "Conn_01x03_Pin"
-			(at 0 7.41 360)
+			(at 0 7.41 0)
 			(layer "F.Fab")
 			(effects
@@
 		(tags "capacitor handsolder")
 		(property "Reference" "C12"
-			(at 3.9 0.14 360)
+			(at 3.9 0.14 0)
 			(layer "F.SilkS")
 			(effects
@@
 		)
 		(property "Value" "10uF"
-			(at 0 1.68 360)
+			(at 0 1.68 0)
 			(layer "F.Fab")
 			(effects
@@
 		)
 		(fp_text user "${REFERENCE}"
-			(at 0 0 360)
+			(at 0 0 0)
 			(layer "F.Fab")
 			(effects
@@
 		(tags "Through hole pin header THT 1x03 2.54mm single row")
 		(property "Reference" "5V1"
-			(at 0 -2.33 360)
+			(at 0 -2.33 0)
 			(layer "F.SilkS")
 			(effects
@@
 		)
 		(property "Value" "Conn_01x03_Pin"
-			(at 0 7.41 360)
+			(at 0 7.41 0)
 			(layer "F.Fab")
 			(effects
@@
 		(tags "capacitor handsolder")
 		(property "Reference" "C5"
-			(at -3 0.2 360)
+			(at -3 0.2 0)
 			(layer "F.SilkS")
 			(effects
@@
 		)
 		(property "Value" "0.1uF"
-			(at 0 1.43 360)
+			(at 0 1.43 0)
 			(layer "F.Fab")
 			(effects
@@
 		)
 		(fp_text user "${REFERENCE}"
-			(at 0 0 360)
+			(at 0 0 0)
 			(layer "F.Fab")
 			(effects
@@
 		(tags "Through hole pin header THT 1x03 2.54mm single row")
 		(property "Reference" "GND1"
-			(at 0 -2.33 360)
+			(at 0 -2.33 0)
 			(layer "F.SilkS")
 			(effects
@@
 		)
 		(property "Value" "Conn_01x03_Pin"
-			(at 0 7.41 360)
+			(at 0 7.41 0)
 			(layer "F.Fab")
 			(effects
@@
 		(tags "capacitor handsolder")
 		(property "Reference" "C10"
-			(at 4.52 -0.4 360)
+			(at 4.52 -0.4 0)
 			(layer "F.SilkS")
 			(effects
@@
 		)
 		(property "Value" "10uF"
-			(at 0 1.68 360)
+			(at 0 1.68 0)
 			(layer "F.Fab")
 			(effects
@@
 		)
 		(fp_text user "${REFERENCE}"
-			(at 0 0 360)
+			(at 0 0 0)
 			(layer "F.Fab")
 			(effects
@@
 		(tags "capacitor handsolder")
 		(property "Reference" "C2"
-			(at 0 -1.43 360)
+			(at 0 -1.43 0)
 			(layer "F.SilkS")
 			(effects
@@
 		)
 		(property "Value" "0.1uF"
-			(at 0 1.43 360)
+			(at 0 1.43 0)
 			(layer "F.Fab")
 			(effects
@@
 		)
 		(fp_text user "${REFERENCE}"
-			(at 0 0 360)
+			(at 0 0 0)
 			(layer "F.Fab")
 			(effects
@@
 		(tags "connector JST PH side entry")
 		(property "Reference" "servo1"
-			(at 2 -2.9 360)
+			(at 2 -2.9 0)
 			(layer "F.SilkS")
 			(hide yes)
@@
 		)
 		(property "Value" "Conn_01x03_Socket"
-			(at 2 4 360)
+			(at 2 4 0)
 			(layer "F.Fab")
 			(effects
@@
 		)
 		(fp_text user "${REFERENCE}"
-			(at 2 1.5 360)
+			(at 2 1.5 0)
 			(layer "F.Fab")
 			(effects
@@
 		)
 		(property "Value" "NC7WZ241K8X"
-			(at 0 0 360)
+			(at 0 0 0)
 			(layer "F.SilkS")
 			(hide yes)
@@
 		)
 		(property "Footprint" "SOP50P310X90-8N"
-			(at 0 0 360)
+			(at 0 0 0)
 			(layer "F.Fab")
 			(hide yes)
@@
 		)
 		(property "Datasheet" "https://componentsearchengine.com/Datasheets/2/NC7WZ241K8X.pdf"
-			(at 0 0 360)
+			(at 0 0 0)
 			(layer "F.Fab")
 			(hide yes)
@@
 		)
 		(property "Description" "Buffers & Line Drivers Dual Buffer with 3-STATE Output"
-			(at 0 0 360)
+			(at 0 0 0)
 			(layer "F.Fab")
 			(hide yes)
@@
 		)
 		(fp_text user "${REFERENCE}"
-			(at 0 0 360)
+			(at 0 0 0)
 			(layer "F.Fab")
 			(effects
@@
 		)
 		(property "Footprint" "DPAK_STM"
-			(at 0 0 360)
+			(at 0 0 0)
 			(layer "F.Fab")
 			(hide yes)
@@
 		)
 		(property "Datasheet" "LD29150DT50R"
-			(at 0 0 360)
+			(at 0 0 0)
 			(layer "F.Fab")
 			(hide yes)
@@
 		)
 		(property "Description" ""
-			(at 0 0 360)
+			(at 0 0 0)
 			(layer "F.Fab")
 			(hide yes)
@@
 		)
 		(fp_text user "*"
-			(at -3.556 6.3881 360)
+			(at -3.556 6.3881 0)
 			(layer "F.SilkS")
 			(effects
@@
 		)
 		(fp_text user "*"
-			(at -2.286 2.8575 360)
+			(at -2.286 2.8575 0)
 			(layer "F.Fab")
 			(effects
@@
 		)
 		(property "Footprint" "DPAK_STM"
-			(at 0 0 360)
+			(at 0 0 0)
 			(layer "F.Fab")
 			(hide yes)
@@
 		)
 		(property "Datasheet" "LD29150DT33R"
-			(at 0 0 360)
+			(at 0 0 0)
 			(layer "F.Fab")
 			(hide yes)
@@
 		)
 		(property "Description" ""
-			(at 0 0 360)
+			(at 0 0 0)
 			(layer "F.Fab")
 			(hide yes)
@@
 		)
 		(fp_text user "*"
-			(at -3.574 7.1481 360)
+			(at -3.574 7.1481 0)
 			(layer "F.SilkS")
 			(effects
@@
 		)
 		(fp_text user "*"
-			(at -2.286 2.8575 360)
+			(at -2.286 2.8575 0)
 			(layer "F.Fab")
 			(effects
@@
 		(tags "resistor handsolder")
 		(property "Reference" "R1"
-			(at -2.2 1.4 360)
+			(at -2.2 1.4 0)
 			(layer "F.SilkS")
 			(effects
@@
 		)
 		(property "Value" "10K"
-			(at 0 1.43 360)
+			(at 0 1.43 0)
 			(layer "F.Fab")
 			(effects
@@
 		)
 		(fp_text user "${REFERENCE}"
-			(at 0 0 360)
+			(at 0 0 0)
 			(layer "F.Fab")
 			(effects
@@
 		)
 		(fp_text user "${REFERENCE}"
-			(at 0 3.81 360)
+			(at 0 3.81 0)
 			(layer "F.Fab")
 			(effects
@@
 		)
 		(fp_text user "${REFERENCE}"
-			(at 0 3.81 360)
+			(at 0 3.81 0)
 			(layer "F.Fab")
 			(effects
@@
 		(tags "nRF24L01 adapter breakout")
 		(property "Reference" "U2"
-			(at 0 -3 360)
+			(at 0 -3 0)
 			(layer "F.SilkS")
 			(effects
@@
 		)
 		(property "Value" "NRF24"
-			(at 13 5 360)
+			(at 13 5 0)
 			(layer "F.Fab")
 			(effects
@@
 		)
 		(fp_text user "${REFERENCE}"
-			(at 12.5 2.5 360)
+			(at 12.5 2.5 0)
 			(layer "F.Fab")
 			(effects
@@
 	)
 	(segment
-		(start 115.075 85)
-		(end 117 85)
-		(width 1)
-		(layer "F.Cu")
-		(net 80)
-	)
-	(segment
 		(start 157.62 81.38)
 		(end 159 80)
@@
 	)
 	(segment
+		(start 116.75 84.75)
+		(end 116.5 85)
+		(width 1)
+		(layer "F.Cu")
+		(net 80)
+	)
+	(segment
 		(start 139 75)
 		(end 138.1125 74.1125)
@@
 	)
 	(segment
+		(start 116.5 85)
+		(end 115.075 85)
+		(width 1)
+		(layer "F.Cu")
+		(net 80)
+	)
+	(segment
 		(start 155.635 86.87)
 		(end 155.0475 86.87)
@@
 	)
 	(via
-		(at 117 85)
+		(at 116.75 84.75)
 		(size 1)
 		(drill 0.3)
@@
 	)
 	(zone
-		(net 3)
-		(net_name "VCC")
+		(net 80)
+		(net_name "GND")
 		(layer "F.Cu")
 		(hatch edge 0.5)
@@
 		(min_thickness 0.25)
 		(filled_areas_thickness no)
-		(fill
+		(fill yes
 			(thermal_gap 0.5)
 			(thermal_bridge_width 0.5)
@@
 			)
 		)
+	)
+	(zone
+		(net 80)
+		(net_name "GND")
+		(layer "B.Cu")
+		(hatch edge 0.5)
+		(priority 3)
+		(connect_pads yes
+			(clearance 0.5)
+		)
+		(min_thickness 0.25)
+		(filled_areas_thickness no)
+		(fill yes
+			(thermal_gap 0.5)
+			(thermal_bridge_width 0.5)
+		)
+		(polygon
+			(pts
+				(xy 107.5 65.5) (xy 108 125.5) (xy 187.5 125.25) (xy 186.5 65)
+			)
+		)

Commit message: not quite sure tbh
Parts:
- Main Terminal: renamed from Main-Terminal1
- moved servo12 12.9 mm to (176.0, 112.2)
- moved servo10 2.95 mm to (176.0, 105.5)
- moved servo2 2.95 mm to (176.0, 78.5)
- moved servo3 2.95 mm to (176.0, 85.0)
- moved servo5 2.95 mm to (176.0, 98.5)
- moved servo7 2.95 mm to (176.0, 91.5)
- renumbered 3.3V1 to 3.3V, 33R1 to 33R, 50R1 to 50R, 5V1 to 5V, GND1 to GND
Routing:
- net Net-(IC2-A2): track 170.6 -> 169.5 mm
Other:
- board text added: "+"
- board text added: "-"
- board text added: "24"
- board text added: "25"
- board text added: "26"
- board text added: "27"
- board text added: "28"
- board text added: "29"
- board text added: "30"
- board text added: "31"
- board text added: "Teensy 4.0 Hexapod Controller"
- board text added: "V0.1"
- board text added: "by Jirakorn Sukmee"
