File: PCB-Teensy4.0/Teensy4.0PCB/Teensy4.0PCB.kicad_sch (KiCad schematic)
At the start: 53 parts, among them IC1 TXB0108PWR, IC2 NC7WZ241K8X, J1 Conn_01x04_Pin, J2 Conn_01x04_Pin, U1 Teensy4.0, U2 NRF24, U3 BNO055

Commit message: not quite sure tbh
Other:
- note added: "JIRAKORN SUKMEE"
- company: (none) -> Jirakorn Sukmee
- title: (none) -> Teensy 4.0 Hexapod Controller
- moved on the sheet: 3.3V1, 5V1, Button1, C2, C3, C4, C5, GND1, R1, R2, R4, R5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
