File: Teensy4.0-PCB/Teensy4.0/Teensy4.0.kicad_sch (KiCad schematic)
At the start: 38 parts, among them IC1 TXB0108PWR, IC2 NC7WZ241K8X, U1 Teensy4.0, U2 NRF24, U3 ICM-20948, U4 TPS62143RGTT

Commit message: updated the PCB 13/01
Parts:
- removed C9: 0.1uF, Capacitor_SMD:C_0805_2012Metric_Pad1.18x1.45mm_HandSolder, symbol Device:C_Small
- removed IC1: TXB0108PWR, SOP65P640X120-20N, symbol TXB0108PWR:TXB0108PWR
- removed U3: ICM-20948, Sensor_Motion:InvenSense_QFN-24_3x3mm_P0.4mm, symbol Sensor_Motion:ICM-20948
- added 5V1, GND1: Conn_01x03_Pin, Connector_PinHeader_2.54mm:PinHeader_1x03_P2.54mm_Vertical, symbol Connector:Conn_01x03_Pin
- added C11, C15, C18, C21, C7: 0.1uF, Capacitor_SMD:C_0805_2012Metric_Pad1.18x1.45mm_HandSolder, symbol Device:C
- added C12, C19, C20, C8: 10uF, Capacitor_SMD:C_0805_2012Metric_Pad1.18x1.45mm_HandSolder, symbol Device:C
- added C13: 470uF, Capacitor_SMD:CP_Elec_10x10, symbol Device:C
- added C14, C9: 47uF, Capacitor_SMD:C_0805_2012Metric_Pad1.18x1.45mm_HandSolder, symbol Device:C
- added C17: 10uF, Capacitor_SMD:C_0805_2012Metric_Pad1.18x1.45mm_HandSolder, symbol Device:C_Small
- added D1: Green, Diode_SMD:D_0805_2012Metric, symbol Device:D
- added D2: RED, Diode_SMD:D_0805_2012Metric, symbol Device:D
- added D3: D, Diode_SMD:D_0805_2012Metric, symbol Device:D
- added D4: BLUE, Diode_SMD:D_0805_2012Metric, symbol Device:D
- added J1: 24-27, Connector_PinHeader_2.54mm:PinHeader_1x04_P2.54mm_Vertical, symbol Connector:Conn_01x04_Pin
- added J2: 28-31, Connector_PinHeader_2.54mm:PinHeader_1x04_P2.54mm_Vertical, symbol Connector:Conn_01x04_Pin
- added Q1, Q2: BSS138, Package_TO_SOT_SMD:SOT-23, symbol Transistor_FET:BSS138
- added Q3: SS8050, Package_TO_SOT_SMD:SOT-23, symbol Transistor_BJT:SS8050
- added R10: 4.66K, Resistor_SMD:R_0805_2012Metric_Pad1.20x1.40mm_HandSolder, symbol Device:R
- added R11, R12, R13: 2.2K, Resistor_SMD:R_0805_2012Metric_Pad1.20x1.40mm_HandSolder, symbol Device:R
- added R2, R3, R4, R5, R8, R9: 10K, Resistor_SMD:R_0805_2012Metric_Pad1.20x1.40mm_HandSolder, symbol Device:R
- added S2: CAN_SERIAL3, Connector_PinHeader_2.54mm:PinHeader_1x02_P2.54mm_Vertical, symbol Connector:Conn_01x02_Pin
- added S3: SERIAL8, Connector_PinHeader_2.54mm:PinHeader_1x02_P2.54mm_Vertical, symbol Connector:Conn_01x02_Pin
- added S4: SERIAL7, Connector_PinHeader_2.54mm:PinHeader_1x02_P2.54mm_Vertical, symbol Connector:Conn_01x02_Pin
- added U3: TXS0104ERGYR, RGY14_2P05X2P05, symbol TXS0104ERGYR:TXS0104ERGYR
- added U5: MIC5504-1.8YM5, Package_TO_SOT_SMD:SOT-23-5, symbol Regulator_Linear:MIC5504-1.8YM5
- added U6: ICM-20948, Sensor_Motion:InvenSense_QFN-24_3x3mm_P0.4mm, symbol Sensor_Motion:ICM-20948
- BZ1: footprint (none) -> Buzzer_Beeper:Buzzer_12x9.5RM7.6
- C1, C2, C3: footprint (none) -> Capacitor_SMD:C_0805_2012Metric_Pad1.18x1.45mm_HandSolder
- C10: footprint Capacitor_SMD:C_0402_1005Metric_Pad0.74x0.62mm_HandSolder -> Capacitor_SMD:C_0805_2012Metric_Pad1.18x1.45mm_HandSolder
- C4: value 22uF / Cer -> 22uF; footprint Capacitor_SMD:C_0402_1005Metric_Pad0.74x0.62mm_HandSolder -> Capacitor_SMD:C_0805_2012Metric_Pad1.18x1.45mm_HandSolder
- C5: value 3.3nF / Cer -> 0.1uF; footprint Capacitor_SMD:C_0402_1005Metric_Pad0.74x0.62mm_HandSolder -> Capacitor_SMD:C_0805_2012Metric_Pad1.18x1.45mm_HandSolder
- C6: value 10uF / Cer -> 10uF; footprint Capacitor_SMD:C_0402_1005Metric_Pad0.74x0.62mm_HandSolder -> Capacitor_SMD:C_0805_2012Metric_Pad1.18x1.45mm_HandSolder
- H1, H2, H3, H4: footprint (none) -> MountingHole:MountingHole_3.2mm_M3
- L1: footprint foorprints4:IND_SRP2512_BRN -> footprints:IND_SRP2512_BRN
- Main-Power1: renamed from Main-Power; footprint (none) -> TerminalBlock_Phoenix:TerminalBlock_Phoenix_MKDS-1,5-2-5.08_1x02_P5.08mm_Horizontal
- R1: value 100k / Film -> 100k; footprint Resistor_SMD:R_0402_1005Metric_Pad0.72x0.64mm_HandSolder -> Resistor_SMD:R_0805_2012Metric_Pad1.20x1.40mm_HandSolder
- R6: value 10K -> 50; footprint Resistor_SMD:R_1206_3216Metric_Pad1.30x1.75mm_HandSolder -> Resistor_SMD:R_0805_2012Metric_Pad1.20x1.40mm_HandSolder
- R7: footprint (none) -> Resistor_SMD:R_0805_2012Metric_Pad1.20x1.40mm_HandSolder
- U1: footprint (none) -> teensy.pretty-master:Teensy40
- button1: renamed from button; footprint (none) -> Button_Switch_THT:SW_PUSH_6mm
Connections:
- net +3V3: now also C14.1, C15.1, C20.2, C21.2, R3.1, R8.1, R9.2, U3.1 (VCCA); no longer R6.1
- net +5V: now also 5V1.1 (Pin_1), 5V1.2 (Pin_2), 5V1.3 (Pin_3), C17.1, C8.1, C9.1, D1.2 (A), U3.14 (VCCB), U5.1 (VIN), U5.3 (EN)
- net GND: now also R6.1, C11.2, C12.2, C13.1, C14.2, C15.2, C17.2, C18.2, C19.2, C20.1, C21.1, C7.1, C8.2, C9.2, GND1.1 (Pin_1), GND1.2 (Pin_2), GND1.3 (Pin_3), Q3.2 (E), R11.1, R12.1, R13.1, U3.15 (EPAD), U3.7 (GND), U5.2 (GND), U6.18 (GND), U6.20 (GND)
- net VCC: now also C13.2, D4.2 (A)
- net servo_dir: now also U3.2 (A1)
- net servo_rx: now also U3.4 (A3)
- net servo_tx: now also U3.3 (A2)
- net at R6.2: now also BZ1.2 (-), D3.1 (K)
- net at IC2.2 (A1): now also U3.12 (B2)
- net at IC2.3 (Y2): now also U3.11 (B3)
- net at IC2.1 (~{OE}), IC2.7 (OE): now also U3.13 (B1)
- net at BZ1.1 (+): now also D3.2 (A), Q3.3 (C)
- net serial_tx2: now reaches U1.10 (8_TX2_IN1)
- net serial_tx2: now also S2.2 (Pin_2)
- net serial_tx3: now reaches U1.21 (14_A0_TX3_SPDIF_OUT)
- net serial_tx3: now also S3.2 (Pin_2)
- net serial_rx3: now reaches U1.22 (15_A1_RX3_SPDIF_IN)
- net serial_rx3: now also S3.1 (Pin_1)
- net serial_rx4: now reaches U1.23 (16_A2_RX4_SCL1)
- net serial_rx4: now also S4.1 (Pin_1)
- net serial_tx4: now reaches U1.24 (17_A3_TX4_SDA1)
- net serial_tx4: now also S4.2 (Pin_2)
- net SDA: now reaches U1.25 (18_A4_SDA0)
- net SDA: now also Q1.3 (D), R3.2
- net SCL: now reaches U1.26 (19_A5_SCL0)
- net SCL: now also Q2.3 (D), R8.2
- net at U1.35 (24_A10_TX6_SCL2): now also J1.1 (Pin_1)
- net at U1.36 (25_A11_RX6_SDA2): now also J1.2 (Pin_2)
- net at U1.37 (26_A12_MOSI1): now also J1.3 (Pin_3)
- net at U1.38 (27_A13_SCK1): now also J1.4 (Pin_4)
- net at U1.39 (28_RX7): now also J2.1 (Pin_1)
- net at U1.40 (29_TX7): now also J2.2 (Pin_2)
- net at U1.41 (30_CRX3): now also J2.3 (Pin_3)
- net at U1.42 (31_CTX3): now also J2.4 (Pin_4)
- net buzzer: now reaches U1.6 (4_BCLK2)
- net buzzer: now also R10.2
- net serial_rx2: now reaches U1.9 (7_RX2_OUT1A)
- net serial_rx2: now also S2.1 (Pin_1)
- net CE renamed NRF_CE
- net CSN renamed NRF_CSN
- net MISO renamed NRF_MISO
- net MOSI renamed NRF_MOSI
- net SCK renamed NRF_SCK
- new net: C7.2, U6.10 (REGOUT)
- new net: R2.2, U6.22 (~{CS})
- new net: Q3.1 (B), R10.1
- new net: D4.1 (K), R13.2
- new net: D1.1 (K), R11.2
- new net: D2.1 (K), R12.2
- new net: R9.1, U3.8 (OE)
- new net +1V8: C11.1, C12.1, C18.1, C19.1, D2.2 (A), Q1.1 (G), Q2.1 (G), R2.1, R4.1, R5.1, U5.5 (VOUT), U6.13 (VDD), U6.8 (VDDIO)
- new net SCL_1V8: Q2.2 (S), R5.2, U6.23 (SCL/SCLK)
- new net SDA_1V8: Q1.2 (S), R4.2, U6.24 (SDA/SDI)
- no-connect marks 11 -> 33
Other:
- note added: "5V -> 1V8 LDO and power LED"
- note added: "Button and Buzzer circuit"
- note added: "ICM-20948 IMU"
- note added: "IMU BIDIRECTIONAL LOGIC CONVERTER 1V8 <-> 3V3"
- note added: "Main Power Bulk Capacitor Mounting Holes"
- note added: "NRF24L01 Module"
- note added: "SERVO CONNECTIONS"
- note added: "SERVO LOGIC CONVERTER"
- note added: "VCC -> 5V Buck Converter"
- title: (none) -> Teensy 4.0 Serial Servo Controller
- moved on the sheet: BZ1, C1, C10, C2, C3, C4, C5, C6, H1, H2, H3, H4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
