File: Teensy4.0-PCB/Teensy4.0/Teensy4.0.kicad_sch (KiCad schematic)
At the start: 75 parts, among them IC2 NC7WZ241K8X, J1 24-27, J2 28-31, Q1 BSS138, Q2 BSS138, Q3 SS8050, U1 Teensy4.0, U2 NRF24, U3 TXS0104ERGYR, U4 TPS62143RGTT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

Commit message: updated some stuff on the PCB
Parts:
- removed Q1, Q2: BSS138, Package_TO_SOT_SMD:SOT-23, symbol Transistor_FET:BSS138
- removed R4, R5, R8: 10K, Resistor_SMD:R_0805_2012Metric_Pad1.20x1.40mm_HandSolder, symbol Device:R
- added C16, C23: 10uF, symbol Device:C
- added C22, C24: 0.1uF, symbol Device:C
- added D5: 3V3 | Red, Diode_SMD:D_0805_2012Metric, symbol Device:D
- added R14: 10K, symbol Device:R
- added U7: TXS0104ERGYR, RGY14_2P05X2P05, symbol TXS0104ERGYR:TXS0104ERGYR
- D1: value Green -> 5V | Green
- D2: value RED -> 1V8
- D4: value BLUE -> VCC
- R11: value 2.2K -> 400
- R12: value 2.2K -> 20
- R13: value 2.2K -> 1.72K
- R3: value 10K -> 300
Connections:
- net +1V8: now also C16.2, C22.1, R14.2, U7.1 (VCCA)
- net +3V3: now also R7.2, C23.2, C24.1, D5.2 (A), U7.14 (VCCB); no longer R3.1
- net +5V: now also R6.1
- net GND: now also R3.1, button1.2, C16.1, C22.2, C23.1, C24.2, U7.15 (EPAD), U7.7 (GND); no longer R6.1, R7.2
- net SCL: now also U7.12 (B2)
- net SCL_1V8: now also U7.3 (A2)
- net SDA: now also U7.13 (B1); no longer R3.2
- net SDA_1V8: now also U7.2 (A1)
- net button: now also R7.1
- net INT_1V8: now reaches U6.12 (INT1)
- net INT_1V8: now also U7.4 (A3)
- net OE_PIN: now reaches IC2.1 (~{OE}), IC2.7 (OE), U3.13 (B1)
- net to_nc7: now reaches IC2.2 (A1), U3.12 (B2)
- net from_nc7: now reaches IC2.3 (Y2), U3.11 (B3)
- net ICM_INT: now reaches U1.27 (20_A6_TX5_LRCLK1)
- net ICM_INT: now also U7.11 (B3)
- new net: R14.1, U7.8 (OE)
- new net: D5.1 (K), R3.2
- no-connect marks 33 -> 35
Other:
- note added: "Green"
- note added: "buzzer not done"
- moved on the sheet: C10, C17, C20, C21, C4, C5, C6, D1, D2, D4, IC2, L1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

Commit message: updated PCB
Parts:
- removed D2: 1V8, Diode_SMD:D_0805_2012Metric, symbol Device:D
- removed Q3: SS8050, Package_TO_SOT_SMD:SOT-23, symbol Transistor_BJT:SS8050
- removed R10: 4.66K, Resistor_SMD:R_0805_2012Metric_Pad1.20x1.40mm_HandSolder, symbol Device:R
- removed R12: 20, Resistor_SMD:R_0805_2012Metric_Pad1.20x1.40mm_HandSolder, symbol Device:R
- removed R6: 50, Resistor_SMD:R_0805_2012Metric_Pad1.20x1.40mm_HandSolder, symbol Device:R
- added R4: 180, Resistor_SMD:R_0805_2012Metric_Pad1.20x1.40mm_HandSolder, symbol Device:R
- added U8: MMBT8099LT1G, SOT-23_ONS, symbol MMBT8099LT1G:MMBT8099LT1G
- C16, C22, C23, C24: footprint (none) -> Capacitor_SMD:C_0805_2012Metric_Pad1.18x1.45mm_HandSolder
- D1, D4, D5: footprint Diode_SMD:D_0805_2012Metric -> Diode_SMD:D_0805_2012Metric_Pad1.15x1.40mm_HandSolder
- D3: value D -> TS4148 RBG; footprint Diode_SMD:D_0805_2012Metric -> Diode_SMD:D_0805_2012Metric_Pad1.15x1.40mm_HandSolder
- R11: value 400 -> 2.2K
- R13: value 1.72K -> 8.2K
- R14: footprint (none) -> Resistor_SMD:R_0805_2012Metric_Pad1.20x1.40mm_HandSolder
- R3: value 300 -> 1.5K
Connections:
- net +5V: now also BZ1.1 (+), D3.1 (K)
- net GND: now also U8.2 (EMITTER)
- net buzzer: now also R4.1
- net at D3.2 (A): now also BZ1.2 (-), U8.3 (COLLECTOR); no longer BZ1.1 (+)
- new net: R4.2, U8.1 (BASE)
Other:
- note added: "might remove LED"
- note added: "should work?"
- note removed: "buzzer not done"
- moved on the sheet: BZ1

Commit message: updated some stuff on the PCB
Parts:
- removed Main-Power1: Screw_Terminal_01x02, TerminalBlock_Phoenix:TerminalBlock_Phoenix_MKDS-1,5-2-5.08_1x02_P5.08mm_Horizontal, symbol Connector:Screw_Terminal_01x02
- added MainPower1: XT30PW-M, footprints:AMASS_XT30PW-M, symbol XT30PW-M:XT30PW-M
- C9: LCSC (none) -> C1713
Connections:
- net GND: now also MainPower1.N
- net VCC: now also MainPower1.P
Changed lines of the file:
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@@
 	(symbol
 		(lib_id "power:GND")
-		(at 364.49 83.82 270)
+		(at 367.03 81.28 270)
 		(unit 1)
 		(exclude_from_sim no)
@@
 		(fields_autoplaced yes)
 		(property "Reference" "#PWR05"
-			(at 358.14 83.82 0)
+			(at 360.68 81.28 0)
 			(effects
 				(font
@@
 		)
 		(property "Value" "GND"
-			(at 360.68 83.8199 90)
+			(at 363.22 81.2799 90)
 			(effects
 				(font
@@
 		)
 		(property "Footprint" ""
-			(at 364.49 83.82 0)
+			(at 367.03 81.28 0)
 			(effects
 				(font
@@
 		)
 		(property "Datasheet" ""
-			(at 364.49 83.82 0)
+			(at 367.03 81.28 0)
 			(effects
 				(font
@@
 		)
 		(property "Description" "Power symbol creates a global label with name \"GND\" , ground"
-			(at 364.49 83.82 0)
+			(at 367.03 81.28 0)
 			(effects
 				(font
@@
 	(symbol
 		(lib_id "power:VCC")
-		(at 364.49 81.28 90)
+		(at 367.03 83.82 90)
 		(unit 1)
 		(exclude_from_sim no)
@@
 		(fields_autoplaced yes)
 		(property "Reference" "#PWR04"
-			(at 368.3 81.28 0)
+			(at 370.84 83.82 0)
 			(effects
 				(font
@@
 		)
 		(property "Value" "VCC"
-			(at 360.68 81.2799 90)
+			(at 363.22 83.8199 90)
 			(effects
 				(font
@@
 		)
 		(property "Footprint" ""
-			(at 364.49 81.28 0)
+			(at 367.03 83.82 0)
 			(effects
 				(font
@@
 		)
 		(property "Datasheet" ""
-			(at 364.49 81.28 0)
+			(at 367.03 83.82 0)
 			(effects
 				(font
@@
 		)
 		(property "Description" "Power symbol creates a global label with name \"VCC\""
-			(at 364.49 81.28 0)
+			(at 367.03 83.82 0)
 			(effects
 				(font
@@
 			)
 		)
+		(property "LCSC" "C1713"
+			(at 92.71 48.26 90)
+			(effects
+				(font
+					(size 1.27 1.27)
+				)
+				(hide yes)
+			)
+		)
 		(pin "1"
 		)
@@
 	)
 	(symbol
+		(lib_id "XT30PW-M:XT30PW-M")
+		(at 372.11 83.82 180)
+		(unit 1)
+		(exclude_from_sim no)
+		(in_bom yes)
+		(on_board yes)
+		(dnp no)
+		(fields_autoplaced yes)
+		(property "Reference" "MainPower1"
+			(at 381 81.2799 0)
+			(effects
+				(font
+					(size 1.27 1.27)
+				)
+				(justify right)
+			)
+		)
+		(property "Value" "XT30PW-M"
+			(at 381 83.8199 0)
+			(effects
+				(font
+					(size 1.27 1.27)
+				)
+				(justify right)
+			)
+		)
+		(property "Footprint" "footprints:AMASS_XT30PW-M"
+			(at 372.11 83.82 0)
+			(effects
+				(font
+					(size 1.27 1.27)
+				)
+				(justify bottom)
+				(hide yes)
+			)
+		)
+		(property "Datasheet" ""
+			(at 372.11 83.82 0)
+			(effects
+				(font
+					(size 1.27 1.27)
+				)
+				(hide yes)
+			)
+		)
+		(property "Description" ""
+			(at 372.11 83.82 0)
+			(effects
+				(font
+					(size 1.27 1.27)
+				)
+				(hide yes)
+			)
+		)
+		(property "MF" "AMASS"
+			(at 372.11 83.82 0)
+			(effects
+				(font
+					(size 1.27 1.27)
+				)
+				(justify bottom)
+				(hide yes)
+			)
+		)
+		(property "MAXIMUM_PACKAGE_HEIGHT" "5 mm"
+			(at 372.11 83.82 0)
+			(effects
+				(font
+					(size 1.27 1.27)
+				)
+				(justify bottom)
+				(hide yes)
+			)
+		)
+		(property "Package" "None"
+			(at 372.11 83.82 0)
+			(effects
+				(font
+					(size 1.27 1.27)
+				)
+				(justify bottom)
+				(hide yes)
+			)
+		)
+		(property "Price" "None"
+			(at 372.11 83.82 0)
+			(effects
+				(font
+					(size 1.27 1.27)
+				)
+				(justify bottom)
+				(hide yes)
+			)
+		)
+		(property "Check_prices" "https://www.snapeda.com/parts/XT30PW-M/AMASS/view-part/?ref=eda"
+			(at 372.11 83.82 0)
+			(effects
+				(font
+					(size 1.27 1.27)
+				)
+				(justify bottom)
+				(hide yes)
+			)
+		)
+		(property "STANDARD" "Manufacturer Recommendations"
+			(at 372.11 83.82 0)
+			(effects
+				(font
+					(size 1.27 1.27)
+				)
+				(justify bottom)
+				(hide yes)
+			)
+		)
+		(property "PARTREV" "1.2"
+			(at 372.11 83.82 0)
+			(effects
+				(font
+					(size 1.27 1.27)
+				)
+				(justify bottom)
+				(hide yes)
+			)
+		)
+		(property "SnapEDA_Link" "https://www.snapeda.com/parts/XT30PW-M/AMASS/view-part/?ref=snap"
+			(at 372.11 83.82 0)
+			(effects
+				(font
+					(size 1.27 1.27)
+				)
+				(justify bottom)
+				(hide yes)
+			)
+		)
+		(property "MP" "XT30PW-M"
+			(at 372.11 83.82 0)
+			(effects
+				(font
+					(size 1.27 1.27)
+				)
+				(justify bottom)
+				(hide yes)
+			)
+		)
+		(property "Description_1" "\n                        \n                            Socket; DC supply; XT30; male; PIN: 2; on PCBs; THT; Colour: yellow\n                        \n"
+			(at 372.11 83.82 0)
+			(effects
+				(font
+					(size 1.27 1.27)
+				)
+				(justify bottom)
+				(hide yes)
+			)
+		)
+		(property "MANUFACTURER" "Amass"
+			(at 372.11 83.82 0)
+			(effects
+				(font
+					(size 1.27 1.27)
+				)
+				(justify bottom)
+				(hide yes)
+			)
+		)
+		(property "Availability" "Not in stock"
+			(at 372.11 83.82 0)
+			(effects
+				(font
+					(size 1.27 1.27)
+				)
+				(justify bottom)
+				(hide yes)
+			)
+		)
+		(property "SNAPEDA_PN" "XT30PW-M"
+			(at 372.11 83.82 0)
+			(effects
+				(font
+					(size 1.27 1.27)
+				)
+				(justify bottom)
+				(hide yes)
+			)
+		)
+		(pin "P"
+		)
+		(pin "N"
+		)
+		(instances
+			(project ""
+				(path "/be95a50c-3bd3-4d52-91b1-8e687e67c64b"
+					(reference "MainPower1")
+					(unit 1)
+				)
+			)
+		)
+	)
+	(symbol
 		(lib_id "Connector:Conn_01x04_Pin")
 		(at 226.06 67.31 180)
@@
 					(unit 1)
 				)
-			)
-		)
-	)
-	(symbol
-		(lib_id "Connector:Screw_Terminal_01x02")
-		(at 369.57 81.28 0)
-		(unit 1)
-		(exclude_from_sim no)
-		(in_bom yes)
-		(on_board yes)
-		(dnp no)
-		(fields_autoplaced yes)
-		(property "Reference" "Main-Power1"
-			(at 372.11 82.5499 0)
-			(effects
-				(font
-					(size 1.27 1.27)
-				)
-				(justify left)
-			)
-		)
-		(property "Value" "Screw_Terminal_01x02"
-			(at 372.11 83.8199 0)
-			(effects
-				(font
-					(size 1.27 1.27)
-				)
-				(justify left)
-				(hide yes)
-			)
-		)
-		(property "Footprint" "TerminalBlock_Phoenix:TerminalBlock_Phoenix_MKDS-1,5-2-5.08_1x02_P5.08mm_Horizontal"
-			(at 369.57 81.28 0)
-			(effects
-				(font
-					(size 1.27 1.27)
-				)
-				(hide yes)
-			)
-		)
-		(property "Datasheet" "~"
-			(at 369.57 81.28 0)
-			(effects
-				(font
-					(size 1.27 1.27)
-				)
-				(hide yes)
-			)
-		)
-		(property "Description" "Generic screw terminal, single row, 01x02, script generated (kicad-library-utils/schlib/autogen/connector/)"
-			(at 369.57 81.28 0)
-			(effects
-				(font
-					(size 1.27 1.27)
-				)
-				(hide yes)
-			)
-		)
-		(pin "2"
-		)
-		(pin "1"
-		)
-		(instances
-			(project ""
-				(path "/be95a50c-3bd3-4d52-91b1-8e687e67c64b"
-					(reference "Main-Power1")
-					(unit 1)
-				)

Commit message: updated pcb: changed from nrf24l01 to lora ra-02
Parts:
- removed U2: NRF24, RF_Module:nRF24L01_Breakout, symbol RF:NRF24L01_Breakout
- added U2: Ai-Thinker-Ra-02, RF_Module:Ai-Thinker-Ra-01-LoRa, symbol RF_Module:Ai-Thinker-Ra-02
- button1: footprint Button_Switch_THT:SW_PUSH_6mm -> Button_Switch_SMD:SW_SPST_PTS647_Sx38
- renumbered D5 to 3V1, D1 to 5V2, D4 to VCC1
Connections:
- net +3V3: now also U2.3 (VDD)
- net GND: now also C13.2, U2.1 (GND), U2.16 (GND), U2.2 (GND), U2.9 (GND); no longer C13.1
- net VCC: now also C13.1; no longer C13.2
- net LORA_IRQ: now reaches U1.8 (6_OUT1D)
- net LORA_IRQ: now also U2.5 (DIO0)
- net NRF_CE renamed LORA_CE
- net LORA_CE: now also U2.4 (~{RESET})
- net NRF_CSN renamed LORA_CSN
- net LORA_CSN: now also U2.15 (~{NSS})
- net NRF_MISO renamed LORA_MISO
- net LORA_MISO: now also U2.13 (MISO)
- net NRF_MOSI renamed LORA_MOSI
- net LORA_MOSI: now also U2.14 (MOSI)
- net NRF_SCK renamed LORA_SCK
- net LORA_SCK: now also U2.12 (SCK)
- no-connect marks 35 -> 37
Other:
- note added: "LoRa RA-02 Module"
- note removed: "NRF24L01 Module"
- note removed: "might remove LED"
- moved on the sheet: 5V1, C15, C3, C9, GND1, S2, S3, S4
