File: Teensy4.0-PCB/Teensy4.0/Teensy4.0.kicad_pcb (KiCad board)
At the start: 4 copper layers, 76 x 58 mm, 75 parts, among them IC2 NC7WZ241K8X, J1 24-27, J2 28-31, Q1 BSS138, Q2 BSS138, Q3 SS8050, U1 Teensy4.0, U2 NRF24, U3 TXS0104ERGYR, U4 TPS62143RGTT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

Commit message: updated PCB
Parts:
- removed D2: RED, Diode_SMD:D_0805_2012Metric
- removed Q1, Q2: BSS138, Package_TO_SOT_SMD:SOT-23
- removed Q3: SS8050, Package_TO_SOT_SMD:SOT-23
- removed R10: 4.66K, Resistor_SMD:R_0805_2012Metric_Pad1.20x1.40mm_HandSolder
- removed R12: 2.2K, Resistor_SMD:R_0805_2012Metric_Pad1.20x1.40mm_HandSolder
- removed R5, R8: 10K, Resistor_SMD:R_0805_2012Metric_Pad1.20x1.40mm_HandSolder
- removed R6: 50, Resistor_SMD:R_0805_2012Metric_Pad1.20x1.40mm_HandSolder
- added 3V3: 3V3 | Red, Diode_SMD:D_0805_2012Metric_Pad1.15x1.40mm_HandSolder, F.Cu at (142.0, 85.2)
- added C16: 10uF, Capacitor_SMD:C_0805_2012Metric_Pad1.18x1.45mm_HandSolder, F.Cu at (144.5, 105.0)
- added C22: 0.1uF, Capacitor_SMD:C_0805_2012Metric_Pad1.18x1.45mm_HandSolder, F.Cu at (146.5, 105.0)
- added C23: 10uF, Capacitor_SMD:C_0805_2012Metric_Pad1.18x1.45mm_HandSolder, F.Cu at (146.5, 101.0)
- added C24: 0.1uF, Capacitor_SMD:C_0805_2012Metric_Pad1.18x1.45mm_HandSolder, F.Cu at (144.5, 101.0)
- added R14: 10K, Resistor_SMD:R_0805_2012Metric_Pad1.20x1.40mm_HandSolder, F.Cu at (150.0, 108.2)
- added U7: TXS0104ERGYR, footprints:RGY14_2P05X2P05, F.Cu at (150.1, 103.1)
- added U8: MMBT8099LT1G, footprints:SOT-23_ONS, F.Cu at (157.7, 111.2)
- 5V: renamed from D1; value Green -> 5V | Green; footprint Diode_SMD:D_0805_2012Metric -> Diode_SMD:D_0805_2012Metric_Pad1.15x1.40mm_HandSolder
- D3: value D -> TS4148 RBG; footprint Diode_SMD:D_0805_2012Metric -> Diode_SMD:D_0805_2012Metric_Pad1.15x1.40mm_HandSolder
- R13: value 2.2K -> 8.2K
- R3: value 10K -> 1.5K
- R4: value 10K -> 180
- VCC: renamed from D4; value BLUE -> VCC; footprint Diode_SMD:D_0805_2012Metric -> Diode_SMD:D_0805_2012Metric_Pad1.15x1.40mm_HandSolder
- moved C8 107.5 mm to (154.3, 86.6)
- moved C11 106.3 mm to (152.1, 92.1), turned to -90 degrees
- moved C12 105.4 mm to (150.1, 92.1), turned to -90 degrees
- moved S2 104.6 mm to (135.9, 84.2), turned to 180 degrees
- moved S3 98.2 mm to (133.0, 84.3), turned to 180 degrees
- moved R4 96.7 mm to (155.8, 108.2)
- moved S4 92.0 mm to (130.1, 84.3), turned to 180 degrees
- moved R3 88.7 mm to (143.0, 89.2), turned to 90 degrees
- moved R13 84.0 mm to (147.5, 89.2), turned to 90 degrees
- moved R11 79.8 mm to (145.2, 89.2), turned to 90 degrees
- moved C3 76.7 mm to (122.2, 112.2)
- moved R9 75.6 mm to (129.5, 120.8), turned to 90 degrees
- moved C14 75.1 mm to (111.8, 87.0), turned to 90 degrees
- moved C9 74.4 mm to (118.5, 87.8)
- moved C15 74.0 mm to (122.2, 114.2)
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Connections:
- net Net-(IC2-A1) renamed /to_nc7
- net Net-(IC2-OE) renamed /OE_PIN
- net Net-(IC2-Y2) renamed /from_nc7
- BZ1 pad 1: Net-(BZ1-+) -> +5V
- D3 pad 1: Net-(BZ1--) -> +5V
- D3 pad 2: Net-(BZ1-+) -> Net-(BZ1--)
- R3 pad 1: +3V3 -> GND
- R3 pad 2: /SDA -> Net-(D5-K)
- R4 pad 1: +1V8 -> /buzzer
- R4 pad 2: /SDA_1V8 -> Net-(U8-BASE)
- R7 pad 1: Net-(R7-Pad1) -> /button
- R7 pad 2: GND -> +3V3
- U1 pad 27: unconnected-(U1-20_A6_TX5_LRCLK1-Pad27) -> /ICM_INT
- U6 pad 12: unconnected-(U6-INT1-Pad12) -> /INT_1V8
- button1 pad 2: Net-(R7-Pad1) -> GND
Routing:
- net GND: track 111.5 -> 228.9 mm, vias 7 -> 14
- net +3V3: track 9.03 -> 76.2 mm, vias 0 -> 3
- net /NRF_SCK: track 0.00 -> 55.6 mm, vias 0 -> 1
- net +5V: track 69.7 -> 111.2 mm
- net /buzzer: track 0.00 -> 36.9 mm, vias 0 -> 1
- net /ICM_INT: track 0.00 -> 34.5 mm, vias 0 -> 2
- net /NRF_MISO: track 0.00 -> 31.3 mm
- net /SCL: track 0.00 -> 31.3 mm, vias 0 -> 1
- net /servo_rx: track 0.00 -> 31.0 mm, vias 0 -> 2
- net /servo_tx: track 0.00 -> 27.6 mm, vias 0 -> 2
- net Net-(IC2-A2): track 73.6 -> 100.2 mm
- net /SDA: track 0.00 -> 26.4 mm, vias 0 -> 1
- net /button: track 0.00 -> 26.3 mm
- net /NRF_MOSI: track 0.00 -> 25.1 mm
- net /servo_dir: track 0.00 -> 24.7 mm, vias 0 -> 2
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- added copper zone on In2.Cu, net GND

Commit message: updated some stuff on the PCB
Parts:
- removed Main-Power1: Screw_Terminal_01x02, TerminalBlock_Phoenix:TerminalBlock_Phoenix_MKDS-1,5-2-5.08_1x02_P5.08mm_Horizontal
- added Main Power: XT30PW-M, footprints:AMASS_XT30PW-M, F.Cu at (164.4, 71.1)
- U4: footprint footprints:RGT16_1P7X1P7 -> footprints3:RGT16_1P7X1P7
- moved servo4 20.8 mm to (163.6, 119.2)
- moved C7 13.5 mm to (152.0, 107.7), turned to 90 degrees
- moved R14 12.7 mm to (154.8, 96.5), turned to -90 degrees
- moved C6 11.6 mm to (124.6, 73.2), turned to -90 degrees
- moved C9 11.5 mm to (109.0, 81.2)
- moved servo2 11.5 mm to (163.6, 113.5)
- moved L1 10.1 mm to (115.7, 73.9), turned to -90 degrees
- moved C4 10.1 mm to (119.2, 71.6), turned to 0 degrees
- moved servo1 9.86 mm to (172.6, 102.2)
- moved servo7 9.85 mm to (172.6, 107.8)
- moved servo9 9.65 mm to (172.6, 91.0)
- moved R2 9.56 mm to (155.8, 99.9), turned to 180 degrees
- moved D3 8.79 mm to (145.2, 113.4)
- moved R1 8.41 mm to (115.4, 77.2), turned to 0 degrees
- moved servo5 7.96 mm to (163.6, 107.8)
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- renumbered 5V1 to 5V, GND1 to GND
Routing:
- net GND: track 228.9 -> 95.8 mm, vias 14 -> 48
- net VCC: track 156.9 -> 74.5 mm, vias 1 -> 0
- net +5V: track 111.2 -> 187.8 mm, vias 5 -> 6
- net +3V3: track 76.2 -> 142.4 mm, vias 3 -> 2
- net Net-(J1-Pin_3): track 0.00 -> 41.4 mm
- net Net-(J1-Pin_4): track 0.00 -> 40.8 mm
- net +1V8: track 35.0 -> 74.3 mm, vias 0 -> 2
- net Net-(J1-Pin_2): track 0.00 -> 37.4 mm
- net Net-(J2-Pin_3): track 0.00 -> 36.3 mm
- net Net-(J2-Pin_4): track 0.00 -> 35.0 mm
- net /serial_rx2: track 0.00 -> 34.6 mm, vias 0 -> 1
- net /serial_tx2: track 0.00 -> 34.6 mm
- net Net-(J2-Pin_2): track 0.00 -> 33.4 mm
- net Net-(J2-Pin_1): track 0.00 -> 28.6 mm, vias 0 -> 2
- net Net-(J1-Pin_1): track 0.00 -> 24.5 mm
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- added copper zone on B.Cu, net GND
- added copper zone on F.Cu, net GND
- added copper zone on In1.Cu, net VCC
Other:
- board text added: "Jirakorn Sukmee's Teensy 4.0 Hexapod Controller"
- board text added: "V0.2"
