File: Teensy4.0-PCB/Teensy4.0/Teensy4.0.kicad_pcb (KiCad board)
At the start: 4 copper layers, 76 x 58 mm, 74 parts, among them IC2 NC7WZ241K8X, J1 24-27, J2 28-31, U1 Teensy4.0, U2 NRF24, U3 TXS0104ERGYR, U4 TPS62143RGTT, U5 MIC5504-1.8YM5, U6 ICM-20948, U7 TXS0104ERGYR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

Commit message: small changes to the PCB
Routing:
- net Net-(IC2-A2): track 105.4 -> 104.0 mm
- net +1V8: track 74.3 -> 75.1 mm
- net GND: track 95.8 -> 95.7 mm, vias 48 -> 51
Changed lines of the file:
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@@
 			(pintype "passive")
 		)
-		(model "/home/jirakorns/Documents/Morphing-Robot/Teensy4.0-PCB/models/US8-8_2P1X2P4_ONS.step"
+		(model "/home/jirakornsukmee/Documents/Morphing-Robot/Teensy4.0-PCB/models/US8-8_2P1X2P4_ONS.step"
 			(offset
 				(xyz 0 0 0)
@@
 			)
 		)
-		(model "/home/jirakorns/Documents/Morphing-Robot/Teensy4.0-PCB/models/ICM-20948.step"
+		(model "/home/jirakornsukmee/Documents/Morphing-Robot/Teensy4.0-PCB/models/ICM-20948.step"
 			(offset
 				(xyz 0 0 0)
@@
 			(pintype "unspecified")
 		)
-		(model "/home/jirakorns/Documents/Morphing-Robot/Teensy4.0-PCB/models/TXS0104ERGYR.step"
+		(model "/home/jirakornsukmee/Documents/Morphing-Robot/Teensy4.0-PCB/models/TXS0104ERGYR.step"
 			(offset
 				(xyz 0 0 0)
@@
 		)
 		(fp_text user "${REFERENCE}"
-			(at 12.5 2.5 0)
+			(at 13.3895 2.325 0)
 			(layer "F.Fab")
 			(effects
@@
 			(pintype "unspecified")
 		)
-		(model "/home/jirakorns/Documents/Morphing-Robot/Teensy4.0-PCB/models/TXS0104ERGYR.step"
+		(model "/home/jirakornsukmee/Documents/Morphing-Robot/Teensy4.0-PCB/models/TXS0104ERGYR.step"
 			(offset
 				(xyz 0 0 0)
@@
 			(pintype "passive")
 		)
-		(model "/home/jirakorns/Documents/Morphing-Robot/Teensy4.0-PCB/models/IND_SRP2512_BRN.step"
+		(model "/home/jirakornsukmee/Documents/Morphing-Robot/Teensy4.0-PCB/models/IND_SRP2512_BRN.step"
 			(offset
 				(xyz 0 0 0)
@@
 			(solder_mask_margin 0.102)
 		)
-		(model "/home/jirakorns/Documents/Morphing-Robot/Teensy4.0-PCB/models/XT30PW-M.step"
+		(model "/home/jirakornsukmee/Documents/Morphing-Robot/Teensy4.0-PCB/models/XT30PW-M.step"
 			(offset
 				(xyz 0 0 0)
@@
 			(pintype "unspecified")
 		)
-		(model "/home/jirakorns/Documents/Morphing-Robot/Teensy4.0-PCB/models/SOT-23_ONS.step"
+		(model "/home/jirakornsukmee/Documents/Morphing-Robot/Teensy4.0-PCB/models/SOT-23_ONS.step"
 			(offset
 				(xyz 0 0 0)
@@
 			(pintype "unspecified")
 		)
-		(model "/home/jirakorns/Documents/Morphing-Robot/Teensy4.0-PCB/models/RGT0016C.stp"
+		(model "/home/jirakornsukmee/Documents/Morphing-Robot/Teensy4.0-PCB/models/RGT0016C.stp"
 			(offset
 				(xyz 0 0 0)
@@
 	)
 	(segment
+		(start 157.3725 101.5)
+		(end 156.81 102.0625)
+		(width 0.3)
+		(layer "F.Cu")
+		(net 5)
+	)
+	(segment
 		(start 119.773592 74.599812)
 		(end 120.523781 75.350001)
@@
 	)
 	(segment
+		(start 158 101.5)
+		(end 157.3725 101.5)
+		(width 0.3)
+		(layer "F.Cu")
+		(net 5)
+	)
+	(segment
 		(start 151.6 85.3125)
 		(end 153.785 85.3125)
@@
 	)
 	(segment
-		(start 156.2475 111.6696)
-		(end 155.3304 111.6696)
-		(width 0.3)
-		(layer "F.Cu")
-		(net 5)
-	)
-	(segment
 		(start 111.25 110)
 		(end 111.25 116.5)
@@
 	)
 	(segment
-		(start 155.3304 111.6696)
-		(end 154.9 112.1)
-		(width 0.3)
-		(layer "F.Cu")
-		(net 5)
-	)
-	(segment
 		(start 158.075 86.75)
 		(end 155.2225 86.75)
@@
 	)
 	(via
-		(at 111.75 70.25)
+		(at 112.5 71)
 		(size 1)
 		(drill 0.3)
@@
 	)
 	(via
+		(at 136.5 124)
+		(size 1)
+		(drill 0.3)
+		(layers "F.Cu" "B.Cu")
+		(free yes)
+		(net 5)
+	)
+	(via
 		(at 128.3 120.7)
 		(size 1)
@@
 	)
 	(via
+		(at 158 101.5)
+		(size 0.6)
+		(drill 0.3)
+		(layers "F.Cu" "B.Cu")
+		(free yes)
+		(net 5)
+	)
+	(via
 		(at 120.373718 80.725002)
 		(size 0.6)
@@
 	)
 	(via
+		(at 159 123)
+		(size 1)
+		(drill 0.3)
+		(layers "F.Cu" "B.Cu")
+		(free yes)
+		(net 5)
+	)
+	(via
 		(at 116.5 124.3)
 		(size 1)
@@
 	)
 	(segment
-		(start 157.13625 104.1375)
-		(end 158.2 103.07375)
-		(width 0.3)
-		(layer "F.Cu")
-		(net 10)
-	)
-	(segment
 		(start 155.8 91.5875)
 		(end 151.6 87.3875)
@@
 	)
 	(segment
-		(start 158.2 93.9875)
-		(end 151.6 87.3875)
+		(start 147.2 98.325)
+		(end 148 98.325)
 		(width 0.3)
 		(layer "F.Cu")
@@
 	)
 	(segment
-		(start 147.2 98.325)
-		(end 148 98.325)
+		(start 145.025 98.3125)
+		(end 144.7125 98.3125)
 		(width 0.3)
 		(layer "F.Cu")
@@
 	)
 	(segment
-		(start 145.025 98.3125)
-		(end 144.7125 98.3125)
+		(start 157.3625 104.1375)
+		(end 159 102.5)
+		(width 0.3)
+		(layer "F.Cu")
+		(net 10)
+	)
+	(segment
+		(start 157 92.7875)
+		(end 151.6 87.3875)
 		(width 0.3)
 		(layer "F.Cu")
@@
 	)
 	(segment
-		(start 158.2 103.07375)
-		(end 158.2 93.9875)
-		(width 0.3)
-		(layer "F.Cu")
-		(net 10)
-	)
-	(segment
 		(start 145.2 98.325)
 		(end 147.2 98.325)
@@
 	)
 	(segment
+		(start 159 102.5)
+		(end 159 99.5)
+		(width 0.3)
+		(layer "F.Cu")
+		(net 10)
+	)
+	(segment
 		(start 148 98.325)
 		(end 148.2 98.125)
@@
 	)
 	(segment
+		(start 159 99.5)
+		(end 157 97.5)
+		(width 0.3)
+		(layer "F.Cu")
+		(net 10)
+	)
+	(segment
 		(start 143.4 97)
 		(end 143.4 96.2)
@@
 	)
 	(segment
+		(start 157 97.5)
+		(end 157 92.7875)
+		(width 0.3)
+		(layer "F.Cu")
+		(net 10)
+	)
+	(segment
 		(start 156.81 104.1375)
-		(end 157.13625 104.1375)
+		(end 157.3625 104.1375)
 		(width 0.3)
 		(layer "F.Cu")
@@
 	)
 	(segment
-		(start 161.25 125.6)
-		(end 143.525 125.6)
+		(start 142.35 124.475)
+		(end 142.35 123.7)
 		(width 0.3)
 		(layer "F.Cu")
@@
 	)
 	(segment
-		(start 167.6 119.25)
-		(end 161.25 125.6)
+		(start 167.6 85.4)
+		(end 167.6 119.25)
 		(width 0.3)
 		(layer "F.Cu")
@@
 	)
 	(segment
-		(start 142.35 124.425)
-		(end 142.35 123.7)
+		(start 167.6 119.25)
+		(end 170.8 119.25)
 		(width 0.3)
 		(layer "F.Cu")
@@
 	)
 	(segment
-		(start 167.6 85.4)
-		(end 167.6 119.25)
+		(start 142.2 125)
+		(end 161.85 125)
 		(width 0.3)
 		(layer "F.Cu")
@@
 	)
 	(segment
-		(start 167.6 119.25)
-		(end 170.8 119.25)
+		(start 141.85 123.7)
+		(end 141.85 124.65)
 		(width 0.3)
 		(layer "F.Cu")
@@
 	)
 	(segment
-		(start 142.8 125.6)
-		(end 143.525 125.6)
-		(width 0.3)
-		(layer "F.Cu")
-		(net 14)
-	)
-	(segment
-		(start 141.85 123.7)
-		(end 141.85 124.65)
+		(start 141.85 124.65)
+		(end 142.2 125)
 		(width 0.3)
 		(layer "F.Cu")
@@
 	)
 	(segment
-		(start 141.85 124.65)
-		(end 142.8 125.6)
+		(start 161.85 125)
+		(end 167.6 119.25)
 		(width 0.3)
 		(layer "F.Cu")
@@
 	)
 	(segment
-		(start 143.525 125.6)
-		(end 142.35 124.425)
+		(start 142.875 125)
+		(end 142.35 124.475)
 		(width 0.3)
 		(layer "F.Cu")

Commit message: updated picutes
Other:
- board text added: "24"
- board text added: "25"
- board text added: "26"
- board text added: "27"
- board text added: "28"
- board text added: "29"
- board text added: "30"
- board text added: "31"
Changed lines of the file:
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@@
 		(layer "Edge.Cuts")
+	)
+	(gr_text "24"
+		(at 136.75 72.5 0)
+		(layer "F.SilkS")
+		(effects
+			(font
+				(size 1 1)
+				(thickness 0.25)
+				(bold yes)
+			)
+			(justify left bottom)
+		)
+	)
+	(gr_text "29"
+		(at 134.25 79.5 0)
+		(layer "F.SilkS")
+		(effects
+			(font
+				(size 1 1)
+				(thickness 0.25)
+				(bold yes)
+			)
+			(justify left bottom)
+		)
+	)
+	(gr_text "31"
+		(at 129 79.5 0)
+		(layer "F.SilkS")
+		(effects
+			(font
+				(size 1 1)
+				(thickness 0.25)
+				(bold yes)
+			)
+			(justify left bottom)
+		)
 	)
 	(gr_text "V0.2"
@@
 		)
 	)
+	(gr_text "26"
+		(at 131.75 72.5 0)
+		(layer "F.SilkS")
+		(effects
+			(font
+				(size 1 1)
+				(thickness 0.25)
+				(bold yes)
+			)
+			(justify left bottom)
+		)
+	)
 	(gr_text "Jirakorn Sukmee's \nTeensy 4.0\nHexapod Controller"
 		(at 109 101.2 0)
@@
 		)
 	)
+	(gr_text "28"
+		(at 136.75 79.5 0)
+		(layer "F.SilkS")
+		(effects
+			(font
+				(size 1 1)
+				(thickness 0.25)
+				(bold yes)
+			)
+			(justify left bottom)
+		)
+	)
+	(gr_text "30"
+		(at 131.75 79.5 0)
+		(layer "F.SilkS")
+		(effects
+			(font
+				(size 1 1)
+				(thickness 0.25)
+				(bold yes)
+			)
+			(justify left bottom)
+		)
+	)
+	(gr_text "25\n"
+		(at 134.25 72.5 0)
+		(layer "F.SilkS")
+		(effects
+			(font
+				(size 1 1)
+				(thickness 0.25)
+				(bold yes)
+			)
+			(justify left bottom)
+		)
+	)
+	(gr_text "27"
+		(at 129 72.5 0)
+		(layer "F.SilkS")
+		(effects
+			(font
+				(size 1 1)
+				(thickness 0.25)
+				(bold yes)
+			)
+			(justify left bottom)
+		)
+	)
 	(dimension
 		(type aligned)
@@
 	)
 	(via
-		(at 122.5 71.55)
-		(size 1)
-		(drill 0.3)
+		(at 122.5 72)
+		(size 1)
+		(drill 0.3)
